Commit message: Add␣wrist␣camera␣and␣teleoperation␣node

File: urdf/arm.urdf.xacro (robot description, xacro)
@@ -13,3 +13,5 @@
     <!-- Camera - commentare per escludere dal modello -->
     <xacro:include filename="armando_camera.urdf.xacro"/>
+    <!-- Camera requested to complete the second task -->
+    <xacro:include filename="my_camera.urdf.xacro"/>
 </robot>

File: urdf/armando_body.urdf.xacro (robot description, xacro)
@@ -396,4 +396,11 @@
     </joint>
     <link name="camera_mount"/>
+    <!-- Frame di montaggio della MIA camera (end-effector) -->
+    <joint name="my_camera_mount_joint" type="fixed">
+        <parent link="crawer_base"/>
+        <child link="my_camera_mount"/>
+        <origin xyz="0.0 0.02 0.01" rpy="1.5708 -1.5708 0"/>
+    </joint>
+    <link name="my_camera_mount"/>
     <!-- ===== Plugin Gazebo ===== -->
     <gazebo>
